File: vfd_igbt_driver/schematics/vfd_igbtdriver.brd (EAGLE design)
At the start: 49.8 x 49.8 mm, 16 parts, among them J1 FS-PW 2,8, J2 FS-PW 2,8, J3 FS-PW 2,8, J4 FS-PW 2,8, J5 FS-P 6,35, J6 FS-P 6,35

Commit message: Multiple Changes
Fixed the footprint bug from the igbt drivers

Added schematics and pcb for dc-bus

Added new folders for partial pfc voltage doubling rectifier

Added schematics for controller
Parts:
- DC1: device dc-dc-converter:NMA -> custom:MGJ2
- moved DC1 3.56 mm to (27.0, 21.7), turned to 0 degrees
- moved C1 3.00 mm to (35.9, 14.9), flipped to the bottom, turned to 180 degrees
- moved C3 1.59 mm to (35.9, 30.2)
- moved C4 1.59 mm to (35.9, 25.1)
Connections:
- net EMITTER: now also DC1.6; no longer DC1.5
- net N$1: now also DC1.5; no longer DC1.4
- net N$2: now also DC1.7; no longer DC1.6
Routing:
- net 0V: track 33.6 -> 39.9 mm, vias 2 -> 1
- net EMITTER: track 73.2 -> 71.1 mm, vias 4 -> 3
- net N$2: track 31.1 -> 32.7 mm, vias 6 -> 5
- net N$1: track 17.8 -> 19.4 mm, vias 4 -> 3
- net +12V: track 33.2 -> 34.5 mm, vias 2 -> 1
Other:
- board size 49.8 x 49.8 mm -> 49.8 x 55.2 mm

Commit message: Updated Schematics
Updated already finnished schematics with Reichelt (DE) parts attribute

Finalized the controller board
Parts:
- removed D3: ZD18, diode:DO35Z10
- added D1: ZD18, diode:DO35Z10
- DC1: value MGJ2D121505SC -> 12V in, +12V -5V out
- J1, J2, J3, J4: value FS-PW 2,8 -> (none)
- J5, J6: value FS-P 6,35 -> (none)
- moved D2 12.7 mm to (32.4, 45.4), turned to 180 degrees
- renumbered OK1 to IC1
Connections:
- net EMITTER: now also D1.C; no longer D2.C
- net GATE: now also D2.C; no longer D3.C
- net N$8: now also D1.A; no longer D3.A
