File: vfd_igbt_driver/schematics/vfd_igbtdriver.brd (EAGLE design)
At the start: 49.8 x 55.2 mm, 16 parts, among them IC1 FOD3120V

Commit message: Minor changes to Schematics Changed IGBT-Driver signal-side connector to plugs Updated Schematic Information Field
Parts:
- removed J1, J2, J3, J4: (no value), con-faston:F061.200
- added U$1: (no value), frames:A4L-LOC
- added X3: JST-XH-04-PIN-LONG-PAD, JST_XH_connnectors:JST-XH-04-PACKAGE-LONG-PAD
Connections:
- net +12V: now also X3.2; no longer J1.1A, J1.1B
- net 0V: now also X3.1; no longer J2.1A, J2.1B
- net CTRL_5V: now also X3.3; no longer J3.1A, J3.1B
- net CTRL_GND: now also X3.4; no longer J4.1A, J4.1B
Routing:
- net CTRL_GND: track 43.4 -> 15.4 mm
- net CTRL_5V: track 28.5 -> 9.46 mm, vias 1 -> 0
- net +12V: track 34.5 -> 20.4 mm
- net 0V: track 39.9 -> 29.3 mm
- net GATE: track 15.7 -> 22.4 mm
Other:
- board size 49.8 x 55.2 mm -> 49.8 x 49.8 mm
- board text added: "(C) 2020 Christoph Klie"
- board text added: "OpenVFD"
- board text added: "VFD IGBT-DRIVER"
- board text added: "Version 1.0"
- board text added: "[1/1]"
