File: vfd_igbt_driver/schematics/vfd_igbtdriver.sch (EAGLE design)
At the start: 16 parts, among them J1 FS-PW 2,8, J2 FS-PW 2,8, J3 FS-PW 2,8, J4 FS-PW 2,8, J5 FS-P 6,35, J6 FS-P 6,35

Commit message: Multiple Changes
Fixed the footprint bug from the igbt drivers

Added schematics and pcb for dc-bus

Added new folders for partial pfc voltage doubling rectifier

Added schematics for controller
Parts:
- DC1: device dc-dc-converter:NMA -> custom:MGJ2

Commit message: Updated Schematics
Updated already finnished schematics with Reichelt (DE) parts attribute

Finalized the controller board
Parts:
- removed D3: ZD18, diode:ZPD
- added D1: ZD18, diode:ZPD
- C1, C3, C4: R (none) -> MKS2-63 470N
- C2: R (none) -> MKS2-63 100N
- D2: R (none) -> ZD18 3W
- DC1: value MGJ2D121505SC -> 12V in, +12V -5V out; R (none) -> MGJ2D121505SC
- J1, J2, J3, J4: value FS-PW 2,8 -> PIN2F061.200; R (none) -> FS-PW 2,8
- J5, J6: value FS-P 6,35 -> PIN2F061.040; R (none) -> FS-P 6,35
- R1: R (none) -> METALL 140
- R2: R (none) -> 2W METALL 15
- renumbered OK1 to IC1
Connections:
- net EMITTER: now also D1.C; no longer D2.C
- net GATE: now also D2.C; no longer D3.C
- net N$8: now also D1.A; no longer D3.A
Other:
- note removed: "2W METALL 15"
- note removed: "MKS2-63 100N"
- note removed: "MKS2-63 470N"
- note removed: "ZD18 3W"
- moved on the sheet: D2

Commit message: Minor changes to Schematics Changed IGBT-Driver signal-side connector to plugs Updated Schematic Information Field
Parts:
- removed J1, J2, J3, J4: PIN2F061.200, con-faston:PIN2F061.200
- added X3: JST-XH-04-PIN-LONG-PAD, JST_XH_connnectors:JST-XH-04-PIN-LONG-PAD
Connections:
- net +12V: now also X3-2.S; no longer J1.1
- net 0V: now also X3-1.S; no longer J2.1
- net CTRL_5V: now also X3-3.S; no longer J3.1
- net CTRL_GND: now also X3-4.S; no longer J4.1
Other:
- note added: "(C) 2020 Christoph Klie"
- note added: "OpenVFD"
- note added: "VFD IGBT DRIVER"
