File: vfd_igbt_driver/schematics/vfd_igbtdriver_brd_production.brd (EAGLE design)
At the start: 160 x 100 mm, 97 parts, among them J1 FS-PW 2,8, J10 FS-PW 2,8, J11 FS-P 6,35, J12 FS-P 6,35, J13 FS-PW 2,8, J14 FS-PW 2,8, J15 FS-PW 2,8, J16 FS-PW 2,8, J17 FS-P 6,35, J18 FS-P 6,35, J19 FS-PW 2,8, J2 FS-PW 2,8, J20 FS-PW 2,8, J21 FS-PW 2,8, J22 FS-PW 2,8, J23 FS-P 6,35, J24 FS-P 6,35, J25 FS-PW 2,8, J26 FS-PW 2,8, J27 FS-PW 2,8, J28 FS-PW 2,8, J29 FS-P 6,35, J3 FS-PW 2,8, J30 FS-P 6,35, J31 FS-PW 2,8, J32 FS-PW 2,8, J33 FS-PW 2,8, J34 FS-PW 2,8, J35 FS-P 6,35, J36 FS-P 6,35, J4 FS-PW 2,8, J5 FS-P 6,35, J6 FS-P 6,35, J7 FS-PW 2,8, J8 FS-PW 2,8, J9 FS-PW 2,8

Commit message: Minor changes to Schematics Changed IGBT-Driver signal-side connector to plugs Updated Schematic Information Field
Parts:
- removed J13, J14, J15, J16, J19, J20, J21, J22, J25, J26, J27, J28, J31, J32, J33, J34: FS-PW 2,8, con-faston:F061.200
- removed J17, J18, J23, J24, J29, J30, J35, J36: FS-P 6,35, con-faston:F061.040
- added X1, X2, X3, X4, X5, X6: JST-XH-04-PIN-LONG-PAD, JST_XH_connnectors:JST-XH-04-PACKAGE-LONG-PAD
- DC1, DC2, DC3, DC4, DC5, DC6: value MGJ2D121505SC -> 12V in, +12V -5V out
- J1, J10, J2, J3, J4, J7, J8, J9: value FS-PW 2,8 -> (none); device con-faston:F061.200 -> con-faston:F061.040
- J11, J12, J5, J6: value FS-P 6,35 -> (none)
- moved J4 123.7 mm to (132.7, 92.4), turned to 180 degrees
- moved J11 107.9 mm to (133.0, 7.62), turned to 0 degrees
- moved J3 103.1 mm to (116.2, 92.4), turned to 180 degrees
- moved J12 91.2 mm to (116.5, 7.62), turned to 0 degrees
- moved J8 85.0 mm to (16.8, 7.62), turned to 0 degrees
- moved J7 68.7 mm to (33.3, 7.62), turned to 0 degrees
- moved J2 58.6 mm to (82.9, 92.4), turned to 180 degrees
- moved J9 52.2 mm to (83.2, 7.62), turned to 0 degrees
- moved J10 50.2 mm to (66.7, 7.62), turned to 0 degrees
- moved J1 49.8 mm to (66.4, 92.4), turned to 180 degrees
- moved D1 49.8 mm to (18.4, 95.6)
- moved D3 37.1 mm to (68.3, 95.6), turned to 0 degrees
- moved D2 12.7 mm to (31.1, 95.6), turned to 180 degrees
- renumbered OK1 to IC1, OK2 to IC2, OK3 to IC3, OK4 to IC4, OK5 to IC5, OK6 to IC6
Connections:
- net +12V: now also X3.2; no longer J1.1A, J1.1B
- net +12V1: now also X1.2; no longer J7.1A, J7.1B
- net +12V2: now also X2.2; no longer J13.1A, J13.1B
- net +12V3: now also X4.2; no longer J19.1A, J19.1B
- net +12V4: now also X5.2; no longer J25.1A, J25.1B
- net +12V5: now also X6.2; no longer J31.1A, J31.1B
- net 0V: now also X3.1; no longer J2.1A, J2.1B
- net 0V1: now also X1.1; no longer J8.1A, J8.1B
- net 0V2: now also X2.1; no longer J14.1A, J14.1B
- net 0V3: now also X4.1; no longer J20.1A, J20.1B
- net 0V4: now also X5.1; no longer J26.1A, J26.1B
- net 0V5: now also X6.1; no longer J32.1A, J32.1B
- net CTRL_5V: now also X3.3; no longer J3.1A, J3.1B
- net CTRL_5V1: now also X1.3; no longer J9.1A, J9.1B
- net CTRL_5V2: now also X2.3; no longer J15.1A, J15.1B
- net CTRL_5V3: now also X4.3; no longer J21.1A, J21.1B
- net CTRL_5V4: now also X5.3; no longer J27.1A, J27.1B
- net CTRL_5V5: now also X6.3; no longer J33.1A, J33.1B
- net CTRL_GND: now also X3.4; no longer J4.1A, J4.1B
- net CTRL_GND1: now also X1.4; no longer J10.1A, J10.1B
- net CTRL_GND2: now also X2.4; no longer J16.1A, J16.1B
- net CTRL_GND3: now also X4.4; no longer J22.1A, J22.1B
- net CTRL_GND4: now also X5.4; no longer J28.1A, J28.1B
- net CTRL_GND5: now also X6.4; no longer J34.1A, J34.1B
- net EMITTER: now also D1.C; no longer D2.C
- net EMITTER1: now also D3.C, J1.A1, J1.A2; no longer D1.C, J11.A1, J11.A2
- net EMITTER2: now also J3.A1, J3.A2; no longer J17.A1, J17.A2
- net EMITTER3: now also J7.A1, J7.A2; no longer J23.A1, J23.A2
- net EMITTER4: now also J9.A1, J9.A2; no longer J29.A1, J29.A2
- net EMITTER5: now also J11.A1, J11.A2; no longer J35.A1, J35.A2
- net GATE: now also D2.C; no longer D3.C
- net GATE1: now also J2.A1, J2.A2; no longer J12.A1, J12.A2
- net GATE2: now also J4.A1, J4.A2; no longer J18.A1, J18.A2
- net GATE3: now also J8.A1, J8.A2; no longer J24.A1, J24.A2
- net GATE4: now also J10.A1, J10.A2; no longer J30.A1, J30.A2
- net GATE5: now also J12.A1, J12.A2; no longer J36.A1, J36.A2
- net N$11: now also D3.A; no longer D1.A
- net N$8: now also D1.A; no longer D3.A
Routing:
- net CTRL_GND2: track 43.4 -> 15.4 mm
- net CTRL_GND1: track 43.4 -> 15.4 mm
- net CTRL_GND: track 43.4 -> 15.4 mm
- net CTRL_GND4: track 43.4 -> 15.4 mm
- net CTRL_GND3: track 43.4 -> 15.4 mm
- net CTRL_GND5: track 43.4 -> 15.4 mm
- net CTRL_5V5: track 28.5 -> 9.46 mm, vias 1 -> 0
- net CTRL_5V2: track 28.5 -> 9.46 mm, vias 1 -> 0
- net CTRL_5V4: track 28.5 -> 9.46 mm, vias 1 -> 0
- net CTRL_5V3: track 28.5 -> 9.46 mm, vias 1 -> 0
- net CTRL_5V: track 28.5 -> 9.46 mm, vias 1 -> 0
- net CTRL_5V1: track 28.5 -> 9.46 mm, vias 1 -> 0
- net +12V2: track 34.5 -> 20.4 mm
- net +12V1: track 34.5 -> 20.4 mm
- net +12V: track 34.5 -> 20.4 mm
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Other:
- outline, holes or cut-outs redrawn
