File: vfd_controller/schematics/vfd_controller.brd (EAGLE design)
At the start: 160 x 100 mm, 83 parts, among them IC10 HCPL-7840, IC11 MPC3201, IC13 MPC3201, IC14 MPC3201, IC15 Atmega1284P, IC2 MAC485, IC4 Attiny861A, IC5 MPC3201, IC6 HCPL-7840, IC7 HCPL-7840, IC9 HCPL-7840, J1 PIN2F061.200, J18 , J19 , J2 PIN2F061.200, J3 PIN2F061.200, J32 , J33 , J4 PIN2F061.200, X1 JST XH2P ST, X10 JST XH4P ST, X11 JST XH4P ST, X12 JST XH4P ST, X13 JST XH4P ST, X14 JST XH4P ST, X2 20MHz, X3 JST XH2P ST, X4 JST XH4P ST, X5 JST XH2P ST, X6 JST XH2P ST, X7 JST XH4P ST, X8 JST XH4P ST, X9 JST XH4P ST

Commit message: Updated Schematics
Updated already finnished schematics with Reichelt (DE) parts attribute

Finalized the controller board
Parts:
- removed C35, C37, C39: 100n, rcl:C025-024X044
- removed IC13, IC14: MPC3201, ic-package:DIL08
- removed J18, J19, J32, J33: (no value), con-faston:F061.200
- removed JP4: (no value), pinhead:1X04
- removed R18, R26, R27: 68R, resistor:0204/5
- added C10, C11, C13: 100n, resistor:C025-024X044
- added C16: 100n, rcl:C025-024X044
- added IC3: MAX 485 CPA, maxim:DIL08
- added IC8: MPC3201, ic-package:DIL08
- added J5, J6, J7, J8: (no value), con-faston:F061.200
- added JP1: 1x6, pinhead:1X06
- added OK1: 6N137, optocoupler:DIL08
- added R1: 10k, rcl:0204V
- added R4: 330R, resistor:0204/7
- added R5: 330R, resistor:0207/12
- added R7: 330R, resistor:0204/5
- added U$1: (no value), frames:A4L-LOC
- added X15, X16, X17: (no value), JST_XH_connnectors:JST-XH-02-PACKAGE-LONG-PAD
- C12: device rcl:C025-024X044 -> resistor:C025-024X044
- C3: value 22p -> 100n
- C4: value 100n -> 22p
- C5: device resistor:C025-024X044 -> rcl:C050-024X044
- C6, C8: device resistor:C025-024X044 -> rcl:C025-024X044
- C7: device resistor:C025-024X044 -> rcl:C025-025X050
- DC1: value MEV1S1205SC -> 12V in, 5V out
- DC2: value (none) -> 5V in, +-5V out
- IC10, IC9: value HCPL-7840 -> MPC3201; device avago:DIL08 -> ic-package:DIL08
- IC2: value MAC485 -> Attiny861A; device maxim:DIL08 -> ic-package:DIL20
- IC4: value Attiny861A -> HCPL-7840; device ic-package:DIL20 -> avago:DIL08
- IC5: value MPC3201 -> HCPL-7840; device ic-package:DIL08 -> avago:DIL08
- J1, J2, J3, J4: value PIN2F061.200 -> (none)
- JP2: value (none) -> 1x4; device pinhead:1X10 -> pinhead:1X04
- JP3: value (none) -> 1x10; device pinhead:1X06 -> pinhead:1X10
- R10, R11: value 330R -> 68R; device resistor:0204/7 -> resistor:0204/5
- R12: value 1k -> 68R
- R2: device rcl:0204/5 -> rcl:0207/12
- R3: value 10k -> 330R; device rcl:0204/5 -> resistor:0204/7
- R6: value 330R -> 1k
- X1: value JST XH2P ST -> 20MHz; device JST_XH_connnectors:JST-XH-02-PACKAGE-LONG-PAD -> IQD-Frequency-Products:HC49
- X10, X11, X12, X13, X7, X8, X9: value JST XH4P ST -> (none)
- X14: value JST XH4P ST -> (none); device JST_XH_connnectors:JST-XH-03-PACKAGE-LONG-PAD -> JST_XH_connnectors:JST-XH-02-PACKAGE-LONG-PAD
- X2: value 20MHz -> (none); device IQD-Frequency-Products:HC49 -> JST_XH_connnectors:JST-XH-02-PACKAGE-LONG-PAD
- X3: value JST XH2P ST -> (none)
- X4: value JST XH4P ST -> (none); device JST_XH_connnectors:JST-XH-04-PACKAGE-LONG-PAD -> JST_XH_connnectors:JST-XH-03-PACKAGE-LONG-PAD
- X5: value JST XH2P ST -> (none); device JST_XH_connnectors:JST-XH-02-PACKAGE-LONG-PAD -> JST_XH_connnectors:JST-XH-03-PACKAGE-LONG-PAD
- X6: value JST XH2P ST -> (none); device JST_XH_connnectors:JST-XH-02-PACKAGE-LONG-PAD -> JST_XH_connnectors:JST-XH-04-PACKAGE-LONG-PAD
- moved C14 137.7 mm to (20.6, 10.8)
- moved R12 135.1 mm to (11.4, 33.7), turned to 180 degrees
- moved IC4 120.6 mm to (23.2, 17.8), turned to 270 degrees
- moved C1 117.2 mm to (80.0, 40.3)
- moved R10 116.3 mm to (11.4, 19.1), turned to 180 degrees
- moved OK4 113.5 mm to (23.2, 50.2), turned to 90 degrees
- moved X4 111.7 mm to (86.4, 7.30), turned to 270 degrees
- moved C15 111.1 mm to (20.6, 25.1), turned to 180 degrees
- moved C9 108.6 mm to (65.4, 63.2), turned to 270 degrees
- moved X3 105.7 mm to (107.6, 5.40), turned to 0 degrees
- moved X6 100.4 mm to (73.7, 8.57), turned to 270 degrees
- moved R11 97.0 mm to (11.4, 16.5), turned to 180 degrees
- moved JP2 96.2 mm to (67.3, 36.8)
- moved X5 95.9 mm to (80.0, 7.30), turned to 270 degrees
- moved X13 83.7 mm to (14.6, 50.5), turned to 90 degrees
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- renumbered C28 to C17, C29 to C18, C30 to C21, C31 to C19, C33 to C20, C34 to C22, C36 to C26, C40 to C23, DC3 to DC2, IC15 to IC1, OK5 to OK2, OK6 to OK3, R19 to R13, R22 to R14, R23 to R15, R24 to R16, R25 to R17
Connections:
- removed net N$35 (its old number): IC10.7, IC14.2
- removed net TEMP1: IC1.40, X13.1
- removed net TEMP2: IC1.39, X14.1
- new net N$15: IC1.34, X4.1
- new net N$16: C7.1, IC1.32
- new net N$23: IC1.39, X3.1
- new net N$24: IC1.40, X2.1
- new net N$32: IC5.7, IC9.2
- new net N$33: OK4.3, R5.2
- new net N$39: OK4.5, X13.3
- new net N$40: OK4.6, X13.2
- new net N$42: OK4.8, X13.1
- new net N$7: IC1.33, X5.1
- new net SW: IC1.18, R5.1
- net +12V: now also C3.1, J1.1A, J1.1B; no longer C1.1, J18.1A, J18.1B
- net +12V-TREIBER: now also J3.1A, J3.1B, X7.3; no longer J32.1A, J32.1B, X4.3
- net +5V: now also C1.1, C10.2, C24.2, C25.2, C27.2, C6.1, C8.1, IC10.1, IC2.15, IC2.5, IC4.8, IC8.1, IC8.8, IC9.1, JP1.5, OK1.8, OK4.2, R1.2, R6.2, X4.2, X5.2, X6.3; no longer C14.1, C35.2, C37.2, C39.2, C4.1, C7.2, C9.1, IC13.1, IC13.8, IC14.1, IC14.8, IC4.15, IC4.5, IC5.1, JP2.5, OK4.8, R12.2, R3.2, X13.2, X14.2, X7.3
- net 0V: now also C3.2, J2.1A, J2.1B; no longer C1.2, J19.1A, J19.1B
- net 0V-TREIBER: now also J4.1A, J4.1B, X7.4; no longer J33.1A, J33.1B, X4.4
- net 232RX: now also JP2.3; no longer JP4.3
- net 232TX: now also JP2.4; no longer JP4.4
- net 485DE: now also R4.1; no longer R11.1
- net 485RX: now also JP2.1, OK1.6, R6.1; no longer JP4.1, OK4.6, R12.1
- net 485TX: now also JP2.2, R3.1; no longer JP4.2, R10.1
- net EN_SVPWM: now also IC1.20, IC2.9, JP3.9; no longer IC1.4, IC4.9, JP2.9
- net GND: now also C1.2, C10.1, C24.1, C25.1, C27.1, C5.2, C6.2, C7.2, C8.2, IC10.3, IC10.4, IC2.16, IC2.6, IC4.5, IC5.5, IC5.6, IC8.3, IC8.4, IC9.3, IC9.4, JP1.6, OK1.5, X2.2, X3.2, X4.3, X5.3, X6.4, X7.2; no longer C12.2, C14.2, C15.2, C3.2, C35.1, C37.1, C39.1, C7.1, IC10.5, IC10.6, IC13.3, IC13.4, IC14.3, IC14.4, IC4.16, IC5.3, IC5.4, IC9.5, IC9.6, JP2.6, OK4.5, X13.3, X14.3, X4.2, X7.4
- net H1: now also IC2.1, JP3.1, X7.1; no longer IC4.1, JP2.1, X12.1
- net H2: now also IC2.3, JP3.3, X9.1; no longer IC4.3, JP2.3, X10.1
- net H3: now also IC2.7, JP3.7, X11.1; no longer IC4.7, JP2.7, X8.1
- net L1: now also IC2.2, JP3.2, X8.1; no longer IC4.2, JP2.2, X11.1
- net L2: now also IC2.4, JP3.4, X10.1; no longer IC4.4, JP2.4, X9.1
- net L3: now also IC2.8, JP3.8, X12.1; no longer IC4.8, JP2.8, X4.1
- net MISO: now also IC2.19, JP1.2; no longer IC4.19, JP3.2
- net MOSI: now also IC2.20, JP1.1; no longer IC4.20, JP3.1
- net N$10: now also IC3.4; no longer IC2.4
- net N$11: now also R4.2; no longer R11.2
- net N$12: now also R3.2; no longer R10.2
- net N$13: now also X16.1; no longer X5.1
- net N$14: now also X16.2; no longer X5.2
- net N$17: now also X15.1; no longer X3.1
- net N$18: now also C14.2, C15.2, C16.2, IC4.4, IC5.4; no longer C24.2, C25.2, C27.2, IC10.4, IC9.4
- net N$19: now also R12.2, X15.2; no longer R18.2, X3.2
- net N$2: now also X6.1; no longer X7.1
- net N$20: now also IC4.2, R10.1; no longer IC6.2, R27.1
- net N$21: now also IC5.2, R12.1; no longer IC7.2, R18.1
- net N$22: now also IC5.3; no longer IC7.3
- net N$25: now also IC6.2; no longer IC9.2
- net N$26: now also IC6.3; no longer IC9.3
- net N$27: now also IC7.2; no longer IC10.2
- net N$28: now also IC7.3; no longer IC10.3
- net N$29: now also C14.1, C15.1, C16.1, IC4.1, IC5.1; no longer C24.1, C25.1, C27.1, IC10.1, IC9.1
- net N$3: now also X6.2; no longer X7.2
- net N$30: now also IC4.3, R11.1; no longer IC6.3, R26.1
- net N$31: now also IC4.7, IC8.2; no longer IC5.2, IC6.7
- net N$34: now also IC10.2, IC6.7; no longer IC13.2, IC9.7
- net N$36: now also R11.2, X14.1; no longer R26.2, X1.1
- net N$37: now also C9.1, IC2.10, JP3.10; no longer C15.1, IC4.10, JP2.10
- net N$38: now also R10.2, X14.2; no longer R27.2, X1.2
- net N$4: now also X17.1; no longer X6.1
- net N$41: now also C5.1, JP1.4, R1.1; no longer C12.1, JP3.4, R3.1
- net N$43: now also X1.1; no longer X2.1
- net N$44: now also C4.1, X1.2; no longer C3.1, X2.2
- net N$5: now also X17.2; no longer X6.2
- net N$6: now also IC3.2, IC3.3; no longer IC2.2, IC2.3
- net N$8: now also IC3.1, R7.2; no longer IC2.1, R6.2
- net N$9: now also OK1.3, R7.1; no longer OK4.3, R6.1
- net RS458_5V: now also C11.1, C12.1, C13.1, IC3.8, J5.1A, J5.1B, OK1.2; no longer C5.1, C6.1, C8.1, IC2.8, J1.1A, J1.1B, OK4.2
- net RS485_A: now also IC3.6, J7.1A, J7.1B; no longer IC2.6, J3.1A, J3.1B
- net RS485_B: now also IC3.7, J6.1A, J6.1B; no longer IC2.7, J2.1A, J2.1B
- net RS485_GND: now also C11.2, C12.2, C13.2, IC3.5, J8.1A, J8.1B; no longer C5.2, C6.2, C8.2, IC2.5, J4.1A, J4.1B
- net SCK: now also IC2.18, JP1.3; no longer IC4.18, JP3.3
- net SENS1: now also IC8.6; no longer IC5.6
- net SENS2: now also IC9.6; no longer IC11.6
- net SENS3: now also IC10.6; no longer IC13.6
- net SENS4: now also IC11.6; no longer IC14.6
- net SENSC: now also IC10.7, IC8.7, IC9.7; no longer IC13.7, IC14.7, IC5.7
- net SENSE: now also IC10.5, IC8.5, IC9.5; no longer IC13.5, IC14.5, IC5.5
- net SS: now also IC2.17; no longer IC4.17
Routing:
- net GND: track 483.4 -> 801.7 mm, vias 2 -> 8
- net +5V: track 434.3 -> 606.8 mm, vias 0 -> 2
- net EN_SVPWM: track 3.49 -> 60.8 mm, vias 0 -> 2
- net +12V-TREIBER: track 31.8 -> 84.0 mm
- net 0V-TREIBER: track 31.8 -> 83.2 mm
- net +12V: track 3.17 -> 41.9 mm
- net SW: track 0.00 -> 37.1 mm, vias 0 -> 2
- net SS: track 0.00 -> 34.9 mm, vias 0 -> 2
- net 0V: track 3.17 -> 34.4 mm
- net TEMP2: track 27.2 -> 0.00 mm
- net N$1: track 0.00 -> 26.7 mm, vias 1 -> 0
- net TEMP1: track 23.4 -> 0.00 mm
- net N$45: track 0.00 -> 21.3 mm
- net SCK: track 4.13 -> 24.1 mm
- net MOSI: track 4.13 -> 24.1 mm
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Other:
- outline, holes or cut-outs redrawn
- board text added: "(C) 2019 Christoph Klie"
- board text added: "VFD-Conroller"
- board text added: "Variable Frequency Drive"
