File: vfd_controller/schematics/vfd_controller.brd (EAGLE design)
At the start: 160 x 100 mm, 90 parts, among them IC1 Atmega1284P, IC10 MPC3201, IC11 MPC3201, IC2 Attiny861A, IC3 MAX 485 CPA, IC4 HCPL-7840, IC5 HCPL-7840, IC6 HCPL-7840, IC7 HCPL-7840, IC8 MPC3201, IC9 MPC3201, J1 , J2 , J3 , J4 , X1 20MHz

Commit message: Updated Parts List and fix Footprint
Fixed 12V to 5V DCDC footprint in Controller PCB

Switched some 100n Capacitor footprints to bigger RM

Updated Parts List
Parts:
- C15, C16, C17, C24, C25, C26, C6: device rcl:C025-024X044 -> rcl:C050-025X075
- C5: device rcl:C050-024X044 -> rcl:C050-025X075
- C7: device rcl:C025-025X050 -> rcl:C025-024X044
- DC1: device dc-dc-converter:NMA -> custom:MEV
- moved DC1 3.86 mm to (123.4, 81.3), turned to 90 degrees
- moved C6 1.27 mm to (117.5, 74.3)
- moved C15 1.27 mm to (19.4, 25.1)
- moved C16 1.27 mm to (19.4, 60.6), flipped to the top, turned to 180 degrees
- moved C17 1.27 mm to (19.4, 74.9)
- moved C24 1.27 mm to (27.0, 25.1)
- moved C25 1.27 mm to (27.0, 60.6)
- moved C26 1.27 mm to (27.0, 74.9)
- moved C7 0.32 mm to (82.5, 14.6)
Connections:
- net +5V: now also DC1.7; no longer DC1.6
Routing:
- net N$18: track 144.1 -> 152.8 mm
- net GND: track 801.7 -> 808.4 mm
- net +12V: track 41.9 -> 43.4 mm
- net +5V: track 606.8 -> 608.3 mm
Other:
- board text added: "Version 1.0"
- board text added: "[1/1]"
