File: vfd_controller/schematics/vfd_controller.sch (EAGLE design)
At the start: 83 parts, among them IC10 HCPL-7840, IC11 MPC3201, IC13 MPC3201, IC14 MPC3201, IC15 Atmega1284P, IC2 MAC485, IC4 Attiny861A, IC5 MPC3201, IC6 HCPL-7840, IC7 HCPL-7840, IC9 HCPL-7840, J1 PIN2F061.200, J18 , J19 , J2 PIN2F061.200, J3 PIN2F061.200, J32 , J33 , J4 PIN2F061.200, X1 JST XH2P ST, X10 JST XH4P ST, X11 JST XH4P ST, X12 JST XH4P ST, X13 JST XH4P ST, X14 JST XH4P ST, X2 20MHz, X3 JST XH2P ST, X4 JST XH4P ST, X5 JST XH2P ST, X6 JST XH2P ST, X7 JST XH4P ST, X8 JST XH4P ST, X9 JST XH4P ST

Commit message: Updated Schematics
Updated already finnished schematics with Reichelt (DE) parts attribute

Finalized the controller board
Parts:
- removed C35, C37, C39: 100n, rcl:C-EU025-024X044
- removed IC13, IC14: MPC3201, ic-package:DIL8
- removed J18, J19, J32, J33: (no value), con-faston:PIN2F061.200
- removed JP4: (no value), pinhead:PINHD-1X4
- removed R18, R26, R27: 68R, resistor:R-EU_0204/5
- added C10, C11, C13: 100n, resistor:C-EU025-024X044
- added C16: 100n, rcl:C-EU025-024X044
- added IC3: MAX 485 CPA, maxim:MAX3468CPA
- added IC8: MPC3201, ic-package:DIL8
- added J5, J6, J7, J8: PIN2F061.200, con-faston:PIN2F061.200
- added JP1: 1x6, pinhead:PINHD-1X6
- added OK1: 6N137, optocoupler:6N137
- added R1: 10k, rcl:R-EU_0204/2V
- added R4: 330R, resistor:R-EU_0204/7
- added R5: 330R, resistor:R-EU_0207/12
- added R7: 330R, resistor:R-EU_0204/5
- added X15, X16, X17: JST-XH-02-PIN-LONG-PAD, JST_XH_connnectors:JST-XH-02-PIN-LONG-PAD
- C1, C14, C15, C17, C22, C23, C24, C25, C26, C27, C9: R (none) -> MKS2-63 100N
- C12: device rcl:C-EU025-024X044 -> resistor:C-EU025-024X044; R (none) -> MKS2-63 100N
- C18, C19, C20, C21: R (none) -> MKS2-63 10N
- C2: R (none) -> KERKO 22p
- C3: value 22p -> 100n; R (none) -> MKS2-63 100N
- C4: value 100n -> 22p; R (none) -> KERKO 22p
- C5: device resistor:C-EU025-024X044 -> rcl:C-EU050-024X044; R (none) -> MKS2-63 100N
- C6, C8: device resistor:C-EU025-024X044 -> rcl:C-EU025-024X044; R (none) -> MKS2-63 100N
- C7: device resistor:C-EU025-024X044 -> rcl:C-EU025-025X050; R (none) -> MKS2-63 100N
- DC1: value MEV1S1205SC -> 12V in, 5V out; R (none) -> MEV1S1205SC
- DC2: value (none) -> 5V in, +-5V out; R (none) -> MEA1D0505SC
- IC1: R (none) -> ATMEGA 1284-P-PU
- IC10, IC9: value HCPL-7840 -> MPC3201; device avago:HCPL-7800 -> ic-package:DIL8; R (none) -> MPC 3201-CI/P
- IC11: R (none) -> MPC 3201-CI/P
- IC2: value MAC485 -> Attiny861A; device maxim:MAX3468CPA -> ic-package:DIL20; R (none) -> ATTINY 861A-PU
- IC4: value Attiny861A -> HCPL-7840; device ic-package:DIL20 -> avago:HCPL-7800
- IC5: value MPC3201 -> HCPL-7840; device ic-package:DIL8 -> avago:HCPL-7800
- J1, J2, J3, J4: value PIN2F061.200 -> (none); R (none) -> FS-PW-6,35
- JP2: value (none) -> 1x4; device pinhead:PINHD-1X10 -> pinhead:PINHD-1X4; R (none) -> MPE 087-1-004
- JP3: value (none) -> 1x10; device pinhead:PINHD-1X6 -> pinhead:PINHD-1X10; R (none) -> MPE 087-1-010
- OK2, OK3, OK4: R (none) -> 6N 137
- R10, R11: value 330R -> 68R; device resistor:R-EU_0204/7 -> resistor:R-EU_0204/5; R (none) -> METALL 68,0
- R12: value 1k -> 68R; R (none) -> METALL 68,0
- R13, R14, R15, R16, R17: R (none) -> METALL 68,0
- R2: device rcl:R-EU_0204/5 -> rcl:R-EU_0207/12; R (none) -> METALL 10,0K
- R3: value 10k -> 330R; device rcl:R-EU_0204/5 -> resistor:R-EU_0204/7; R (none) -> METALL 330
- R6: value 330R -> 1k; R (none) -> METALL 1,00K
- R8, R9: R (none) -> METALL 1,00K
- X1: value JST XH2P ST -> 20MHz; device JST_XH_connnectors:JST-XH-02-PIN-LONG-PAD -> IQD-Frequency-Products:CRYSTALS-NOGND-HC49; R (none) -> 20,0000-HC49U-S
- X10, X11, X12, X7, X8, X9: value JST XH4P ST -> JST-XH-04-PIN-LONG-PAD; R (none) -> JST XH4P ST
- X13: value JST XH4P ST -> JST-XH-03-PIN-LONG-PAD; R (none) -> JST XH3P ST
- X14: value JST XH4P ST -> JST-XH-02-PIN-LONG-PAD; device JST_XH_connnectors:JST-XH-03-PIN-LONG-PAD -> JST_XH_connnectors:JST-XH-02-PIN-LONG-PAD; R (none) -> JST XH2P ST
- X2: value 20MHz -> JST-XH-02-PIN-LONG-PAD; device IQD-Frequency-Products:CRYSTALS-NOGND-HC49 -> JST_XH_connnectors:JST-XH-02-PIN-LONG-PAD; R (none) -> JST XH2P ST
- X3: value JST XH2P ST -> JST-XH-02-PIN-LONG-PAD; R (none) -> JST XH2P ST
- X4: value JST XH4P ST -> JST-XH-03-PIN-LONG-PAD; device JST_XH_connnectors:JST-XH-04-PIN-LONG-PAD -> JST_XH_connnectors:JST-XH-03-PIN-LONG-PAD; R (none) -> JST XH3P ST
- X5: value JST XH2P ST -> JST-XH-03-PIN-LONG-PAD; device JST_XH_connnectors:JST-XH-02-PIN-LONG-PAD -> JST_XH_connnectors:JST-XH-03-PIN-LONG-PAD; R (none) -> JST XH3P ST
- X6: value JST XH2P ST -> JST-XH-04-PIN-LONG-PAD; device JST_XH_connnectors:JST-XH-02-PIN-LONG-PAD -> JST_XH_connnectors:JST-XH-04-PIN-LONG-PAD; R (none) -> JST XH4P ST
- renumbered C28 to C17, C29 to C18, C30 to C21, C31 to C19, C33 to C20, C34 to C22, C36 to C26, C40 to C23, DC3 to DC2, IC15 to IC1, OK5 to OK2, OK6 to OK3, R19 to R13, R22 to R14, R23 to R15, R24 to R16, R25 to R17
Connections:
- removed net N$35 (its old number): IC10.VOUT+, IC14.2
- removed net TEMP1: IC1.40, X13-1.S
- removed net TEMP2: IC1.39, X14-1.S
- new net N$15: IC1.34, X4-1.S
- new net N$16: C7.1, IC1.32
- new net N$23: IC1.39, X3-1.S
- new net N$24: IC1.40, X2-1.S
- new net N$32: IC5.VOUT+, IC9.2
- new net N$33: OK4.C, R5.2
- new net N$39: OK4.GND, X13-3.S
- new net N$40: OK4.VO, X13-2.S
- new net N$42: OK4.VCC, X13-1.S
- new net N$7: IC1.33, X5-1.S
- new net SW: IC1.18, R5.1
- net +12V: now also C3.1, J1.1; no longer C1.1, J18.1
- net +12V-TREIBER: now also J3.1, X7-3.S; no longer J32.1, X4-3.S
- net +5V: now also C1.1, C10.2, C24.2, C25.2, C27.2, C6.1, C8.1, IC10.1, IC10.8, IC2.15, IC2.5, IC4.VDD2, IC5.VDD2, IC8.1, IC8.8, IC9.1, IC9.8, JP1.5, OK1.VCC, OK4.A, R1.2, R6.2, X4-2.S, X5-2.S, X6-3.S; no longer C14.1, C35.2, C37.2, C39.2, C4.1, C7.2, C9.1, IC10.VDD2, IC13.1, IC13.8, IC14.1, IC14.8, IC4.15, IC4.5, IC5.1, IC5.8, IC9.VDD2, JP2.5, OK4.VCC, R12.2, R3.2, X13-2.S, X14-2.S, X7-3.S
- net 0V: now also C3.2, J2.1; no longer C1.2, J19.1
- net 0V-TREIBER: now also J4.1, X7-4.S; no longer J33.1, X4-4.S
- net 232RX: now also JP2.3; no longer JP4.3
- net 232TX: now also JP2.4; no longer JP4.4
- net 485DE: now also R4.1; no longer R11.1
- net 485RX: now also JP2.1, OK1.VO, R6.1; no longer JP4.1, OK4.VO, R12.1
- net 485TX: now also JP2.2, R3.1; no longer JP4.2, R10.1
- net EN_SVPWM: now also IC1.20, IC2.9, JP3.9; no longer IC1.4, IC4.9, JP2.9
- net GND: now also C1.2, C10.1, C24.1, C25.1, C27.1, C5.2, C6.2, C7.2, C8.2, IC10.3, IC10.4, IC2.16, IC2.6, IC4.GND2, IC4.VOUT-, IC5.GND2, IC5.VOUT-, IC8.3, IC8.4, IC9.3, IC9.4, JP1.6, OK1.GND, X2-2.S, X3-2.S, X4-3.S, X5-3.S, X6-4.S, X7-2.S; no longer C12.2, C14.2, C15.2, C3.2, C35.1, C37.1, C39.1, C7.1, IC10.GND2, IC10.VOUT-, IC13.3, IC13.4, IC14.3, IC14.4, IC4.16, IC4.6, IC5.3, IC5.4, IC9.GND2, IC9.VOUT-, JP2.6, OK4.GND, X13-3.S, X14-3.S, X4-2.S, X7-4.S
- net H1: now also IC2.1, JP3.1, X7-1.S; no longer IC4.1, JP2.1, X12-1.S
- net H2: now also IC2.3, JP3.3, X9-1.S; no longer IC4.3, JP2.3, X10-1.S
- net H3: now also IC2.7, JP3.7, X11-1.S; no longer IC4.7, JP2.7, X8-1.S
- net L1: now also IC2.2, JP3.2, X8-1.S; no longer IC4.2, JP2.2, X11-1.S
- net L2: now also IC2.4, JP3.4, X10-1.S; no longer IC4.4, JP2.4, X9-1.S
- net L3: now also IC2.8, JP3.8, X12-1.S; no longer IC4.8, JP2.8, X4-1.S
- net MISO: now also IC2.19, JP1.2; no longer IC4.19, JP3.2
- net MOSI: now also IC2.20, JP1.1; no longer IC4.20, JP3.1
- net N$10: now also IC3.DI; no longer IC2.DI
- net N$11: now also R4.2; no longer R11.2
- net N$12: now also R3.2; no longer R10.2
- net N$13: now also X16-1.S; no longer X5-1.S
- net N$14: now also X16-2.S; no longer X5-2.S
- net N$17: now also X15-1.S; no longer X3-1.S
- net N$18: now also C14.2, C15.2, C16.2, IC4.GND1, IC5.GND1; no longer C24.2, C25.2, C27.2, IC10.GND1, IC9.GND1
- net N$19: now also R12.2, X15-2.S; no longer R18.2, X3-2.S
- net N$2: now also X6-1.S; no longer X7-1.S
- net N$20: now also IC4.VIN+, R10.1; no longer IC6.VIN+, R27.1
- net N$21: now also IC5.VIN+, R12.1; no longer IC7.VIN+, R18.1
- net N$22: now also IC5.VIN-; no longer IC7.VIN-
- net N$25: now also IC6.VIN+; no longer IC9.VIN+
- net N$26: now also IC6.VIN-; no longer IC9.VIN-
- net N$27: now also IC7.VIN+; no longer IC10.VIN+
- net N$28: now also IC7.VIN-; no longer IC10.VIN-
- net N$29: now also C14.1, C15.1, C16.1, IC4.VDD1, IC5.VDD1; no longer C24.1, C25.1, C27.1, IC10.VDD1, IC9.VDD1
- net N$3: now also X6-2.S; no longer X7-2.S
- net N$30: now also IC4.VIN-, R11.1; no longer IC6.VIN-, R26.1
- net N$31: now also IC4.VOUT+, IC8.2; no longer IC5.2, IC6.VOUT+
- net N$34: now also IC10.2, IC6.VOUT+; no longer IC13.2, IC9.VOUT+
- net N$36: now also R11.2, X14-1.S; no longer R26.2, X1-1.S
- net N$37: now also C9.1, IC2.10, JP3.10; no longer C15.1, IC4.10, JP2.10
- net N$38: now also R10.2, X14-2.S; no longer R27.2, X1-2.S
- net N$4: now also X17-1.S; no longer X6-1.S
- net N$41: now also C5.1, JP1.4, R1.1; no longer C12.1, JP3.4, R3.1
- net N$43: now also X1.1; no longer X2.1
- net N$44: now also C4.1, X1.2; no longer C3.1, X2.2
- net N$5: now also X17-2.S; no longer X6-2.S
- net N$6: now also IC3.DE, IC3.RE/; no longer IC2.DE, IC2.RE/
- net N$8: now also IC3.RO, R7.2; no longer IC2.RO, R6.2
- net N$9: now also OK1.C, R7.1; no longer OK4.C, R6.1
- net RS458_5V: now also C11.1, C12.1, C13.1, IC3.VCC, J5.1, OK1.A; no longer C5.1, C6.1, C8.1, IC2.VCC, J1.1, OK4.A
- net RS485_A: now also IC3.A, J7.1; no longer IC2.A, J3.1
- net RS485_B: now also IC3.B, J6.1; no longer IC2.B, J2.1
- net RS485_GND: now also C11.2, C12.2, C13.2, IC3.GND, J8.1; no longer C5.2, C6.2, C8.2, IC2.GND, J4.1
- net SCK: now also IC2.18, JP1.3; no longer IC4.18, JP3.3
- net SENS1: now also IC8.6; no longer IC5.6
- net SENS2: now also IC9.6; no longer IC11.6
- net SENS3: now also IC10.6; no longer IC13.6
- net SENS4: now also IC11.6; no longer IC14.6
- net SENSC: now also IC10.7, IC8.7, IC9.7; no longer IC13.7, IC14.7, IC5.7
- net SENSE: now also IC10.5, IC8.5, IC9.5; no longer IC13.5, IC14.5, IC5.5
- net SS: now also IC2.17; no longer IC4.17

Commit message: Updated Parts List and fix Footprint
Fixed 12V to 5V DCDC footprint in Controller PCB

Switched some 100n Capacitor footprints to bigger RM

Updated Parts List
Parts:
- C1, C10, C11, C12, C13, C14, C22, C23, C27, C3, C8, C9: R MKS2-63 100N -> MKS02-63 100N
- C15, C16, C17, C24, C25, C26, C6: device rcl:C-EU025-024X044 -> rcl:C-EU050-025X075
- C18, C19, C20, C21: R MKS2-63 10N -> MKS02-63 10N
- C5: device rcl:C-EU050-024X044 -> rcl:C-EU050-025X075
- C7: device rcl:C-EU025-025X050 -> rcl:C-EU025-024X044; R MKS2-63 100N -> MKS02-63 100N
- DC1: device dc-dc-converter:NMA -> custom:MEV
