File: vfd_controller/schematics/vfd_controller_cpu.brd (EAGLE design)
At the start: 107.3 x 100 mm, 36 parts, among them IC1 Atmega1284P, IC2 Attiny861A, J1 , J2 , X1 20MHz, X13 JST-XH-07-PIN-LONG-PAD, X5 JST-XH-10-PIN-LONG-PAD, X6 JST-XH-02-PIN-LONG-PAD

Commit message: Minor changes to Schematics Changed IGBT-Driver signal-side connector to plugs Updated Schematic Information Field
Other:
- board text added: "OpenVFD"
- board text removed: "Variable Frequency Drive"
Changed lines of the file:
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@@
 <hole x="86.95055" y="50.62855" drill="3.2" locked="yes"/>
 <hole x="124.09805" y="50.62855" drill="3.2" locked="yes"/>
-<text x="168.75125" y="18.415" size="2.54" layer="48">Variable Frequency Drive</text>
-<text x="167.66056875" y="13.335" size="2.54" layer="48">VFD-Conroller CPU Board</text>
-<text x="170.23294375" y="8.255" size="2.54" layer="48">(C) 2020 Christoph Klie</text>
+<text x="180.49875" y="17.78" size="2.54" layer="48">OpenVFD</text>
+<text x="167.66056875" y="13.0175" size="2.54" layer="48">VFD-Conroller CPU Board</text>
+<text x="170.23294375" y="7.9375" size="2.54" layer="48">(C) 2020 Christoph Klie</text>
 <circle x="86.9696" y="137.7061" radius="0.762" width="0.508" layer="16"/>
 <circle x="124.1044" y="137.7061" radius="0.762" width="0.508" layer="16"/>
