File: vfd_controller/schematics/vfd_controller_io.brd (EAGLE design)
At the start: 52.4 x 100 mm, 24 parts, among them IC1 HCPL-7840, IC2 HCPL-7840, IC3 MPC3201, IC4 MPC3201, IC5 MPC3201, IC6 MPC3201, X3 JST-XH-03-PIN-LONG-PAD, X4 JST-XH-03-PIN-LONG-PAD, X5 JST-XH-10-PIN-LONG-PAD, X6 JST-XH-02-PIN-LONG-PAD, X7 JST-XH-02-PIN-LONG-PAD

Commit message: Minor changes to Schematics Changed IGBT-Driver signal-side connector to plugs Updated Schematic Information Field
Other:
- board text added: "OpenVFD"
- board text removed: "Variable Frequency Drive"
Changed lines of the file:
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@@
 <hole x="110.617" y="56.34355" drill="3.2"/>
 <hole x="147.7645" y="56.34355" drill="3.2"/>
-<text x="168.11625" y="18.415" size="2.54" layer="48">Variable Frequency Drive</text>
-<text x="168.61306875" y="13.335" size="2.54" layer="48">VFD-Conroller I/O Board</text>
-<text x="169.59794375" y="8.255" size="2.54" layer="48">(C) 2020 Christoph Klie</text>
+<text x="180.18125" y="17.78" size="2.54" layer="48">OpenVFD</text>
+<text x="168.61306875" y="13.0175" size="2.54" layer="48">VFD-Conroller I/O Board</text>
+<text x="169.59794375" y="7.9375" size="2.54" layer="48">(C) 2020 Christoph Klie</text>
 <circle x="110.5916" y="143.4211" radius="0.762" width="0.508" layer="16"/>
 <circle x="147.7772" y="143.4211" radius="0.762" width="0.508" layer="16"/>
