File: vfd_dcbus/schematics/vfd_dcbus.brd (EAGLE design)
At the start: 160 x 100 mm, 44 parts, among them J10 VT FS-P 6,35, J11 VT FS-P 6,35, J12 VT FS-P 6,35, J13 VT FS-PW 6,35, J14 VT FS-P 6,35, J15 VT FS-P 6,35, J16 VT FS-PW 6,35, J17 VT FS-P 6,35, J18 VT FS-P 6,35, J19 VT FS-P 6,35, J20 VT FS-P 6,35, J21 VT FS-P 6,35, J22 VT FS-P 6,35, J23 VT FS-P 6,35, J24 VT FS-P 6,35, J25 VT FS-PW 6,35, J26 VT FS-P 6,35, J27 VT FS-P 6,35, J28 VT FS-P 6,35, J29 VT FS-P 6,35, J3 VT FS-PW 6,35, J30 VT FS-P 6,35, J31 VT FS-P 6,35, J4 VT FS-P 6,35, J5 VT FS-P 6,35, J6 VT FS-PW 6,35, J7 VT FS-P 6,35, J8 VT FS-P 6,35, J9 VT FS-P 6,35

Commit message: Update Controller Schematic & PCB
Parts:
- added U$1: (no value), frames:A4L-LOC
- added X1, X2, X3, X4, X5: JST XH2P ST, JST_XH_connnectors:JST-XH-02-PACKAGE-LONG-PAD
- R1, R2, R4, R5: device rcl:0207/7 -> rcl:0207/5V
- moved R3 4.98 mm to (69.4, 49.9)
- moved R2 1.68 mm to (67.6, 46.1), turned to 90 degrees
- moved R4 1.64 mm to (67.6, 53.7), turned to 270 degrees
- moved J6 1.59 mm to (149.2, 13.0)
- moved R11 1.27 mm to (18.1, 69.2)
- moved R17 1.27 mm to (18.1, 30.8)
- moved R1 1.01 mm to (70.6, 41.0), turned to 270 degrees
- moved J25 0.95 mm to (149.2, 22.9)
- moved R5 0.91 mm to (70.6, 58.9)
- moved J13 0.16 mm to (10.8, 50.0)
- moved R15 0.16 mm to (32.1, 50.0)
Connections:
- removed net N$5: R4.2, R5.1
- new net N$2: R4.1, R5.1
- net DC+: now also R1.2; no longer R1.1
- net DC-: now also X1.2
- net DC--: now also X1.1
- net N$1: now also R1.1; no longer R1.2
- net U_IN: now also X2.2
- net U_MEAS+: now also X5.1
- net U_MEAS-: now also R4.2, X5.2; no longer R4.1
- net U_OUT: now also X2.1
- net V_IN: now also X3.2
- net V_OUT: now also X3.1
- net W_IN: now also X4.1
- net W_OUT: now also X4.2
Routing:
- net DC-: track 89.9 -> 109.4 mm, vias 1 -> 0
- net DC--: track 163.1 -> 181.3 mm, vias 1 -> 0
- net U_MEAS+: track 20.4 -> 5.08 mm, vias 1 -> 0
- net U_MEAS-: track 16.7 -> 5.08 mm, vias 1 -> 0
- net V_IN: track 0.00 -> 7.04 mm, vias 1 -> 0
- net U_IN: track 0.00 -> 7.04 mm, vias 1 -> 0
- net W_IN: track 0.00 -> 6.60 mm, vias 1 -> 0
- net W_OUT: track 0.00 -> 6.16 mm, vias 1 -> 0
- net V_OUT: track 0.00 -> 6.16 mm, vias 1 -> 0
- net U_OUT: track 0.00 -> 5.27 mm, vias 1 -> 0
- net N$2: track 0.00 -> 3.04 mm
- net N$5: track 1.59 -> 0.00 mm
- net N$1: track 1.59 -> 3.15 mm
Other:
- outline, holes or cut-outs redrawn
- board text added: "(C) 2019 Christoph Klie"
- board text added: "DC-BUS"
- board text added: "Variable Frequency Drive"
- board text added: "Version 1.0"
- board text added: "[1/1]"

Commit message: Updated Schematics
Updated already finnished schematics with Reichelt (DE) parts attribute

Finalized the controller board
Parts:
- removed J30, J31: VT FS-P 6,35, con-faston:F061.080
- removed R11, R15: ISA SMT R010-1, resistor:R2512
- added J1: (no value), con-faston:F061.200
- added J2: (no value), con-faston:F061.080
- added R6, R8: 470k, rcl:0207/5V
- C1, C2, C3, C4, C5, C6: value BE LXS 120/450 -> 120µ
- J10, J11, J12, J14, J15, J17, J19, J20, J21, J22, J23, J24, J26, J27, J28, J5, J7, J8, J9: value VT FS-P 6,35 -> (none)
- J13: value VT FS-PW 6,35 -> (none)
- J16, J25, J3, J6: value VT FS-PW 6,35 -> (none); device con-faston:F061.200 -> con-faston:F061.080
- J18, J29, J4: value VT FS-P 6,35 -> (none); device con-faston:F061.080 -> con-faston:F061.200
- R1, R4: value MPR 470K -> 10m; device rcl:0207/5V -> resistor:R2512
- R2: value MPR 470K -> 470k
- R3: value SPR-1206 470 -> 470k; device rcl:R1206 -> rcl:0207/5V
- R5: value MPR 470K -> 470R; device rcl:0207/5V -> rcl:R1206
- R7, R9: value ISA SMT R010-1 -> 10m
- X1, X2, X3, X4, X5: value JST XH2P ST -> (none)
- moved J4 137.7 mm to (149.2, 13.0)
- moved X1 134.6 mm to (18.0, 66.1), turned to 0 degrees
- moved J25 124.1 mm to (25.1, 22.2), turned to 180 degrees
- moved J29 115.1 mm to (149.2, 22.9)
- moved X5 93.1 mm to (151.7, 82.3), turned to 270 degrees
- moved J6 85.6 mm to (64.1, 22.5), turned to 180 degrees
- moved J23 72.4 mm to (64.1, 88.3)
- moved J5 72.1 mm to (25.1, 88.3)
- moved J9 72.1 mm to (25.1, 77.8)
- moved J18 67.1 mm to (10.8, 37.1)
- moved J3 63.9 mm to (64.1, 27.6)
- moved J19 63.8 mm to (25.1, 16.8), turned to 0 degrees
- moved J21 63.6 mm to (25.1, 11.7)
- moved J27 61.0 mm to (25.1, 27.3)
- moved R1 59.6 mm to (18.1, 69.2), flipped to the bottom, turned to 0 degrees
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- renumbered C18 to C1, C19 to C2, C20 to C3, C21 to C4, C22 to C5, C23 to C6, R12 to R9, R17 to R7
Connections:
- net DC+: now also J3.1A, J3.1B, J4.1A, J4.1B, R2.2; no longer J5.1A, J5.1B, J9.1A, J9.1B, R1.2
- net DC-: now also J29.1A, J29.1B, X5.2; no longer J25.1A, J25.1B, X1.2
- net DC--: now also J23.1A, J23.1B, J26.1A, J26.1B, J28.1A, J28.1B, R8.2, X5.1; no longer J18.1A, J18.1B, J19.1A, J19.1B, J21.1A, J21.1B, R5.2, X1.1
- net N$1: now also R3.1; no longer R1.1
- net N$2: now also R6.1, R8.1; no longer R4.1, R5.1
- net U_IN: now also J2.1A, J2.1B, J5.1A, J5.1B, J9.1A, J9.1B, R1.1, X1.2; no longer J26.1A, J26.1B, J27.1A, J27.1B, J4.1A, J4.1B, R11.1, X2.2
- net U_MEAS+: now also R3.2, R5.1, X4.1; no longer R2.2, R3.1, X5.1
- net U_MEAS-: now also R5.2, R6.2, X4.2; no longer R3.2, R4.2, X5.2
- net U_OUT: now also J1.1A, J1.1B, R1.2, X1.1; no longer J3.1A, J3.1B, R11.2, X2.1
- net V_IN: now also J16.1A, J16.1B, J17.1A, J17.1B, R4.1, X2.2; no longer J28.1A, J28.1B, J29.1A, J29.1B, R15.1, X3.2
- net V_OUT: now also R4.2, X2.1; no longer R15.2, X3.1
- net W_IN: now also J19.1A, J19.1B, J21.1A, J21.1B, J25.1A, J25.1B, J27.1A, J27.1B, X3.1; no longer J17.1A, J17.1B, J23.1A, J23.1B, J30.1A, J30.1B, J31.1A, J31.1B, X4.1
- net W_OUT: now also J18.1A, J18.1B, X3.2; no longer J16.1A, J16.1B, X4.2
Routing:
- net N$6: track 0.00 -> 17.1 mm
- net N$3: track 0.45 -> 15.9 mm
- net N$5: track 0.00 -> 14.9 mm
- net N$4: track 0.00 -> 14.0 mm
Other:
- outline, holes or cut-outs redrawn
