File: vfd_dcbus/schematics/vfd_dcbus.brd (EAGLE design)
At the start: 160 x 100 mm, 50 parts

Commit message: Minor changes to Schematics Changed IGBT-Driver signal-side connector to plugs Updated Schematic Information Field
Other:
- board text added: "OpenVFD"
- board text removed: "Variable Frequency Drive"
